File: motor-control-brain-board.kicad_sch (KiCad schematic)
At the start: 35 parts, among them J1 GPIO, J10 PWM, J11 PWR, J12 POWER_SENSE, J13 MISC_SENSE, J2 I2C, J3 SERIAL_1, J4 SERIAL_2, J5 CAN, J6 SPI, J7 USB_C_Receptacle_USB2.0_16P, J8 SWD, J9 POS_SENSE, SW1 RST, U1 TLV76750QWDRBxQ1, U2 TLV76733QWDRBxQ1

Commit message: Routing
Connections:
- net LPUART1_RX: now also J3.3 (Pin_3); no longer J3.4 (Pin_4)
- net LPUART1_TX: now also J3.4 (Pin_4); no longer J3.3 (Pin_3)
- net UART2_RX: now also J4.3 (Pin_3); no longer J4.4 (Pin_4)
- net UART2_TX: now also J4.4 (Pin_4); no longer J4.3 (Pin_3)
Changed lines of the file:
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@@
 	)
 	(junction
+		(at 83.82 163.83)
+		(diameter 0)
+		(color 0 0 0 0)
+	)
+	(junction
 		(at 231.14 27.94)
 		(diameter 0)
@@
 	)
 	(junction
-		(at 83.82 161.29)
-		(diameter 0)
-		(color 0 0 0 0)
-	)
-	(junction
 		(at 92.71 21.59)
 		(diameter 0)
@@
 	(wire
 		(pts
-			(xy 83.82 161.29) (xy 99.06 161.29)
-		)
-		(stroke
-			(width 0)
-			(type default)
-		)
-	)
-	(wire
-		(pts
 			(xy 83.82 60.96) (xy 59.69 60.96)
 		)
@@
 	(wire
 		(pts
-			(xy 33.02 163.83) (xy 99.06 163.83)
+			(xy 33.02 163.83) (xy 83.82 163.83)
 		)
 		(stroke
@@
 	(wire
 		(pts
-			(xy 83.82 161.29) (xy 83.82 173.99)
+			(xy 81.28 171.45) (xy 99.06 171.45)
 		)
 		(stroke
@@
 	(wire
 		(pts
-			(xy 81.28 171.45) (xy 99.06 171.45)
+			(xy 232.41 17.78) (xy 232.41 27.94)
 		)
 		(stroke
@@
 	(wire
 		(pts
-			(xy 232.41 17.78) (xy 232.41 27.94)
+			(xy 83.82 163.83) (xy 99.06 163.83)
 		)
 		(stroke
@@
 	(wire
 		(pts
-			(xy 33.02 161.29) (xy 83.82 161.29)
+			(xy 33.02 161.29) (xy 99.06 161.29)
 		)
 		(stroke
@@
 	(wire
 		(pts
+			(xy 83.82 163.83) (xy 83.82 173.99)
+		)
+		(stroke
+			(width 0)
+			(type default)
+		)
+	)
+	(wire
+		(pts
 			(xy 241.3 27.94) (xy 242.57 27.94)
 		)
@@
 		)
 	)
-	(label "LPUART1_TX"
+	(label "LPUART1_RX"
 		(at 93.98 143.51 180)
 		(effects
@@
 		)
 	)
-	(label "UART2_TX"
+	(label "UART2_RX"
 		(at 93.98 161.29 180)
 		(effects
@@
 		)
 	)
-	(label "UART2_RX"
+	(label "UART2_TX"
 		(at 93.98 163.83 180)
 		(effects
@@
 		)
 	)
-	(label "LPUART1_RX"
+	(label "LPUART1_TX"
 		(at 93.98 146.05 180)
 		(effects
@@
 			)
 		)
-		(pin "USART2_RX" input
-			(at 99.06 163.83 180)
-			(effects
-				(font
-					(size 1.27 1.27)
-				)
-				(justify left)
-			)
-		)
-		(pin "USART2_TX" input
-			(at 99.06 161.29 180)
-			(effects
-				(font
-					(size 1.27 1.27)
-				)
-				(justify left)
-			)
-		)
 		(pin "HRTIM1_CHE2" input
 			(at 137.16 78.74 0)
@@
 			)
 		)
-		(pin "LPUART1_RX" input
-			(at 99.06 146.05 180)
-			(effects
-				(font
-					(size 1.27 1.27)
-				)
-				(justify left)
-			)
-		)
-		(pin "LPUART1_TX" input
-			(at 99.06 143.51 180)
-			(effects
-				(font
-					(size 1.27 1.27)
-				)
-				(justify left)
-			)
-		)
 		(pin "GPIO_PC15" input
 			(at 99.06 78.74 180)
@@
 			(effects
 				(font
+					(size 1.27 1.27)
+				)
+				(justify left)
+			)
+		)
+		(pin "LPUART1_RX" input
+			(at 99.06 143.51 180)
+			(effects
+				(font
+					(size 1.27 1.27)
+				)
+				(justify left)
+			)
+		)
+		(pin "LPUART1_TX" input
+			(at 99.06 146.05 180)
+			(effects
+				(font
+					(size 1.27 1.27)
+				)
+				(justify left)
+			)
+		)
+		(pin "USART2_RX" input
+			(at 99.06 161.29 180)
+			(effects
+				(font
+					(size 1.27 1.27)
+				)
+				(justify left)
+			)
+		)
+		(pin "USART2_TX" input
+			(at 99.06 163.83 180)
+			(effects
+				(font

Commit message: Adjusted cap sizes, 0603 for all need hand soldering, 0402 where possible, 0804 as needed
Parts:
- C2, C3, C5, C6, C7: footprint Capacitor_SMD:C_0402_1005Metric -> Capacitor_SMD:C_0603_1608Metric
- C4: footprint Capacitor_SMD:C_0402_1005Metric -> Capacitor_SMD:C_0805_2012Metric
- U1, U2: footprint Package_SON:VSON-8-1EP_3x3mm_P0.65mm_EP1.65x2.4mm -> Package_SON:VSON-8-1EP_3x3mm_P0.65mm_EP1.65x2.4mm_ThermalVias
Changed lines of the file:
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@@
 			)
 		)
-		(property "Footprint" "Capacitor_SMD:C_0402_1005Metric"
+		(property "Footprint" "Capacitor_SMD:C_0603_1608Metric"
 			(at 237.1852 38.1 0)
 			(effects
@@
 			)
 		)
-		(property "Footprint" "Capacitor_SMD:C_0402_1005Metric"
+		(property "Footprint" "Capacitor_SMD:C_0603_1608Metric"
 			(at 93.6752 30.48 0)
 			(effects
@@
 			)
 		)
-		(property "Footprint" "Capacitor_SMD:C_0402_1005Metric"
+		(property "Footprint" "Capacitor_SMD:C_0603_1608Metric"
 			(at 243.5352 63.5 0)
 			(effects
@@
 			)
 		)
-		(property "Footprint" "Capacitor_SMD:C_0402_1005Metric"
+		(property "Footprint" "Capacitor_SMD:C_0603_1608Metric"
 			(at 209.2452 38.1 0)
 			(effects
@@
 			)
 		)
-		(property "Footprint" "Capacitor_SMD:C_0402_1005Metric"
+		(property "Footprint" "Capacitor_SMD:C_0805_2012Metric"
 			(at 235.9152 63.5 0)
 			(effects
@@
 			)
 		)
-		(property "Footprint" "Package_SON:VSON-8-1EP_3x3mm_P0.65mm_EP1.65x2.4mm"
+		(property "Footprint" "Package_SON:VSON-8-1EP_3x3mm_P0.65mm_EP1.65x2.4mm_ThermalVias"
 			(at 250.19 19.05 0)
 			(effects
@@
 			)
 		)
-		(property "Footprint" "Capacitor_SMD:C_0402_1005Metric"
+		(property "Footprint" "Capacitor_SMD:C_0603_1608Metric"
 			(at 265.1252 38.1 0)
 			(effects
@@
 			)
 		)
-		(property "Footprint" "Package_SON:VSON-8-1EP_3x3mm_P0.65mm_EP1.65x2.4mm"
+		(property "Footprint" "Package_SON:VSON-8-1EP_3x3mm_P0.65mm_EP1.65x2.4mm_ThermalVias"
 			(at 222.25 19.05 0)
 			(effects
